Commit message: 添加摄像头插件配置，修改 camera.urdf.xacro 和 sensor_plugin.xacro

File: base_robot_ws/src/base_robot/urdf/4_robot/plugins/sensor_plugin.xacro (robot description, xacro)
@@ -110,4 +110,29 @@
             </sensor>
         </gazebo>
+<gazebo reference="camera_link">
+    <sensor type="depth" name="camera_sensor">
+        <plugin name="depth_camera" filename="libgazebo_ros_camera.so">
+            <frame_name>camera_optical_link</frame_name>
+        </plugin>
+        <always_on>true</always_on>
+        <update_rate>10</update_rate>
+        <camera name="camera">
+            <horizontal_fov>1.5009831567</horizontal_fov>
+            <image>
+                <width>800</width>
+                <height>600</height>
+                <format>R8G8B8</format>
+            </image>
+            <distortion>
+                <k1>0.0</k1>
+                <k2>0.0</k2>
+                <k3>0.0</k3>
+                <p1>0.0</p1>
+                <p2>0.0</p2>
+                <center>0.5 0.5</center>
+            </distortion>
+        </camera>
+    </sensor>
+</gazebo>
     </xacro:macro>
 </robot>

File: base_robot_ws/src/base_robot/urdf/4_robot/sensor/camera.urdf.xacro (robot description, xacro)
@@ -1,22 +1,37 @@
 <?xml version="1.0"?>
-<robot xmlns:xacro="http://www.ros.org/wiki.xacro">
+<robot xmlns:xacro="http://www.ros.org/wiki/xacro">
     <xacro:macro name="camera_xacro" params="xyz">
-        <!--camera-->
+        <!-- ============相机模块================ -->
         <link name="camera_link">
             <visual>
-                <origin xyz="0.0 0.0 0.0" rpy="0.0 0.0 0.0"/>
+                <origin xyz="0 0 0.0" rpy="0 0 0" />
                 <geometry>
-                    <box size="0.02 0.10 0.02"/>
+                    <box size="0.02 0.10 0.02" />
                 </geometry>
                 <material name="black">
-                    <color rgba="0.0 0.0 0.0 0.5"/>
+                    <color rgba="0.0 0.0 0.0 0.8"/>
                 </material>
             </visual>
+            <collision>
+                <origin xyz="0 0 0.0" rpy="0 0 0" />
+                <geometry>
+                    <box size="0.02 0.10 0.02" />
+                </geometry>
+                <material name="black">
+                    <color rgba="0.0 0.0 0.0 0.8"/>
+                </material>
+            </collision>
+            <xacro:box_inertia m="0.01" w="0.02" h="0.10" d="0.02" />
         </link>
-        <!--机器人关节-->
-        <joint name="camera_link_joint" type="fixed">
-            <parent link="base_link"/>
-            <child link="camera_link"/>
-            <origin xyz="${xyz}" rpy="0.0 0.0 0.0"/>
+        <link name="camera_optical_link"></link>
+        <joint name="camera_optical_joint" type="fixed">
+            <parent link="camera_link" />
+            <child link="camera_optical_link" />
+            <origin xyz="0 0 0" rpy="${-pi/2} 0 ${-pi/2}" />
+        </joint>
+        <joint name="camera_joint" type="fixed">
+            <parent link="base_link" />
+            <child link="camera_link" />
+            <origin xyz="${xyz}" />
         </joint>
     </xacro:macro>
