Commit message: feat: 添加夹爪抓取修复插件，增强底盘控制，完善文档与仓库维护
**新增功能：**
- 新增 gazebo_grasp_plugin 包，以 fixed joint 方案根治 Gazebo ODE 仿真中夹爪穿模/弹飞/打滑问题
- simple_commander.py 新增底盘线速度/角速度 GUI 滑块控制
- auto_task.py 重构为基于 gz topic 持久订阅的附着检测抓取任务流程

**优化改进：**
- arm.xacro: 夹爪手指高摩擦参数(μ=10.0)+关节阻尼配置+gazebo_grasp_fix插件
- test.world: 清理仿真运行时状态块，添加机器人初始位姿及抓取插件配置
- Launch.md: 全文重写，新增系统前置要求、包结构说明、完整依赖清单、一键安装命令、常见问题排查
- README.md: 重构为项目主README，新增V1.2.0版本日志及快速开始指南
- .gitignore: 新增 VS Code db 缓存、Claude Code 工作目录忽略规则

**新增文件：**
- gazebo_grasp_plugin/ (C++ Model Plugin，约1250行源码)
- 夹爪抓取问题分析与修复方案.md (技术文档)

Co-Authored-By: Claude Opus 4.8 <noreply@anthropic.com>

File: base_robot_ws/src/base_robot/urdf/4_robot/arm.xacro (robot description, xacro)
@@ -205,5 +205,6 @@
         <child link="link7" />
         <axis xyz="0 0 -1" />
-        <limit lower="0" upper="0.04" effort="10" velocity="1" />
+        <limit lower="0" upper="0.04" effort="5" velocity="1" />
+        <dynamics damping="10" friction="5"/>
     </joint>
     <link name="link8">
@@ -231,5 +232,6 @@
         <child link="link8" />
         <axis xyz="0 0 1" />
-        <limit lower="-0.04" upper="0" effort="10" velocity="1" />
+        <limit lower="-0.04" upper="0" effort="5" velocity="1" />
+        <dynamics damping="10" friction="5"/>
     </joint>
     <xacro:macro name="gazebo_link" params="ref">
@@ -246,4 +248,23 @@
     <xacro:gazebo_link ref="link5"/>
     <xacro:gazebo_link ref="link6"/>
+    <!-- 夹爪手指高摩擦 + 软接触参数，防止打滑和抖动 -->
+    <gazebo reference="link7">
+        <self_collide>false</self_collide>
+        <mu1>10.0</mu1>
+        <mu2>10.0</mu2>
+        <kp>10000</kp>
+        <kd>500</kd>
+        <minDepth>0.005</minDepth>
+        <maxVel>0.5</maxVel>
+    </gazebo>
+    <gazebo reference="link8">
+        <self_collide>false</self_collide>
+        <mu1>10.0</mu1>
+        <mu2>10.0</mu2>
+        <kp>10000</kp>
+        <kd>500</kd>
+        <minDepth>0.005</minDepth>
+        <maxVel>0.5</maxVel>
+    </gazebo>
     <ros2_control name="GazeboSimSystem" type="system">
         <hardware>
@@ -273,3 +294,20 @@
         </plugin>
     </gazebo>
+    <gazebo>
+        <plugin name="gazebo_grasp_fix" filename="libgazebo_grasp_fix.so">
+            <arm>
+                <arm_name>default_arm</arm_name>
+                <palm_link>link6</palm_link>
+                <gripper_link>link7</gripper_link>
+                <gripper_link>link8</gripper_link>
+            </arm>
+            <forces_angle_tolerance>90</forces_angle_tolerance>
+            <update_rate>50</update_rate>
+            <grip_count_threshold>1</grip_count_threshold>
+            <max_grip_count>10</max_grip_count>
+            <release_tolerance>0.01</release_tolerance>
+            <disable_collisions_on_attach>true</disable_collisions_on_attach>
+            <contact_topic>__default_topic__</contact_topic>
+        </plugin>
+    </gazebo>
 </robot>
