Commit message: 新增导航地图、wrist_camera配置、auto_task脚本、kdl_parser模块及世界文件
Co-Authored-By: Claude Opus 4.7 <noreply@anthropic.com>

File: base_robot_ws/src/base_robot/urdf/4_robot/4_robot.urdf.xacro (robot description, xacro)
@@ -34,5 +34,5 @@
     <xacro:imu_xacro xyz="0 0 0.02"/>
     <xacro:laser_xacro xyz="0 0 0.10"/>
-    <xacro:camera_xacro xyz="0.09 0 0.07"/>
+    <xacro:camera_xacro xyz="-0.03 0.0 0.06" parent_link="link6" rpy="${-pi} ${-pi/2} 0"/>
     <xacro:microphone_xacro xyz="0.15 0 0.08"/>
     <xacro:gazebo_sensor_plugin/>

File: base_robot_ws/src/base_robot/urdf/4_robot/base_robot.urdf.xacro (robot description, xacro)
@@ -29,5 +29,5 @@
             <parent link="base_footprint"/>
             <child link="base_link"/>
-            <origin xyz="0 0 ${length/2.0+0.032-0.001}" rpy="0 0 0"/>
+            <origin xyz="0 0 ${length/2.0+0.05}" rpy="0 0 0"/>
         </joint>
     </xacro:macro>

File: base_robot_ws/src/base_robot/urdf/4_robot/plugins/sensor_plugin.xacro (robot description, xacro)
@@ -135,4 +135,29 @@
     </sensor>
 </gazebo> -->
+    <gazebo reference="wrist_camera_link">
+        <sensor type="depth" name="wrist_camera_sensor">
+            <plugin name="wrist_depth_camera" filename="libgazebo_ros_camera.so">
+                <frame_name>wrist_camera_optical_link</frame_name>
+            </plugin>
+            <always_on>true</always_on>
+            <update_rate>10</update_rate>
+            <camera name="wrist_camera">
+                <horizontal_fov>1.5009831567</horizontal_fov>
+                <image>
+                    <width>640</width>
+                    <height>480</height>
+                    <format>R8G8B8</format>
+                </image>
+                <distortion>
+                    <k1>0.0</k1>
+                    <k2>0.0</k2>
+                    <k3>0.0</k3>
+                    <p1>0.0</p1>
+                    <p2>0.0</p2>
+                    <center>0.5 0.5</center>
+                </distortion>
+            </camera>
+        </sensor>
+    </gazebo>
     </xacro:macro>
 </robot>

File: base_robot_ws/src/base_robot/urdf/4_robot/sensor/camera.urdf.xacro (robot description, xacro)
@@ -1,14 +1,14 @@
 <?xml version="1.0"?>
 <robot xmlns:xacro="http://www.ros.org/wiki/xacro">
-    <xacro:macro name="camera_xacro" params="xyz">
-        <!-- ============相机模块================ -->
+    <xacro:macro name="camera_xacro" params="xyz parent_link:=base_link rpy:='0 0 0'">
+        <!-- ============相机模块 - 缩小一半的小正方体================ -->
         <link name="camera_link">
             <visual>
                 <origin xyz="0 0 0.0" rpy="0 0 0" />
                 <geometry>
-                    <box size="0.02 0.10 0.02" />
+                    <box size="0.0125 0.0125 0.0125" />
                 </geometry>
-                <material name="black">
-                    <color rgba="0.0 0.0 0.0 0.8"/>
+                <material name="red">
+                    <color rgba="1.0 0.0 0.0 1.0"/>
                 </material>
             </visual>
@@ -16,11 +16,11 @@
                 <origin xyz="0 0 0.0" rpy="0 0 0" />
                 <geometry>
-                    <box size="0.02 0.10 0.02" />
+                    <box size="0.0125 0.0125 0.0125" />
                 </geometry>
-                <material name="black">
-                    <color rgba="0.0 0.0 0.0 0.8"/>
+                <material name="red">
+                    <color rgba="1.0 0.0 0.0 1.0"/>
                 </material>
             </collision>
-            <xacro:box_inertia m="0.01" w="0.02" h="0.10" d="0.02" />
+            <xacro:box_inertia m="0.0025" w="0.0125" h="0.0125" d="0.0125" />
         </link>
         <link name="camera_optical_link"></link>
@@ -31,7 +31,7 @@
         </joint>
         <joint name="camera_joint" type="fixed">
-            <parent link="base_link" />
+            <parent link="${parent_link}" />
             <child link="camera_link" />
-            <origin xyz="${xyz}" />
+            <origin xyz="${xyz}" rpy="${rpy}" />
         </joint>
     </xacro:macro>

Commit message: 新增底盘前置深度相机（front_camera_sensor），修复 world 内 mesh 绝对路径
- camera.urdf.xacro 宏增加 prefix 参数，支持多相机实例（默认命名不变）
- 底盘前端顶部 (x=0.22, 离地 0.176m) 挂载水平朝前的 800x600 深度相机
- demo_scene.world / test.world 内嵌模型同步加入相机传感器与外观
- 话题：/front_camera_sensor/image_raw、depth/image_raw、points
- world 内 38 处 /home/lhy 绝对路径改为本机工作空间路径

Co-Authored-By: Claude Opus 4.7 <noreply@anthropic.com>

File: base_robot_ws/src/base_robot/urdf/4_robot/4_robot.urdf.xacro (robot description, xacro)
@@ -35,4 +35,6 @@
     <xacro:laser_xacro xyz="0 0 0.10"/>
     <xacro:camera_xacro xyz="-0.03 0.0 0.06" parent_link="link6" rpy="${-pi} ${-pi/2} 0"/>
+    <!-- 前置相机：底盘前端顶部、水平朝前（离地约 0.176m），用于观察前方路面与墙壁 -->
+    <xacro:camera_xacro xyz="0.22 0 0.06625" parent_link="base_link" rpy="0 0 0" prefix="front_camera"/>
     <xacro:microphone_xacro xyz="0.15 0 0.08"/>
     <xacro:gazebo_sensor_plugin/>

File: base_robot_ws/src/base_robot/urdf/4_robot/plugins/sensor_plugin.xacro (robot description, xacro)
@@ -135,4 +135,30 @@
     </sensor>
 </gazebo> -->
+    <!-- 前置相机（底盘前端，水平朝前）：与腕部相机同为 depth 类型，话题前缀 /front_camera_sensor -->
+    <gazebo reference="front_camera_link">
+        <sensor type="depth" name="front_camera_sensor">
+            <plugin name="front_depth_camera" filename="libgazebo_ros_camera.so">
+                <frame_name>front_camera_optical_link</frame_name>
+            </plugin>
+            <always_on>true</always_on>
+            <update_rate>10</update_rate>
+            <camera name="front_camera">
+                <horizontal_fov>1.5009831567</horizontal_fov>
+                <image>
+                    <width>800</width>
+                    <height>600</height>
+                    <format>R8G8B8</format>
+                </image>
+                <distortion>
+                    <k1>0.0</k1>
+                    <k2>0.0</k2>
+                    <k3>0.0</k3>
+                    <p1>0.0</p1>
+                    <p2>0.0</p2>
+                    <center>0.5 0.5</center>
+                </distortion>
+            </camera>
+        </sensor>
+    </gazebo>
     <gazebo reference="wrist_camera_link">
         <sensor type="depth" name="wrist_camera_sensor">

File: base_robot_ws/src/base_robot/urdf/4_robot/sensor/camera.urdf.xacro (robot description, xacro)
@@ -1,7 +1,8 @@
 <?xml version="1.0"?>
 <robot xmlns:xacro="http://www.ros.org/wiki/xacro">
-    <xacro:macro name="camera_xacro" params="xyz parent_link:=base_link rpy:='0 0 0'">
+    <!-- prefix 用于区分多个相机实例（默认 camera，保持原有命名不变；前置相机传 front_camera） -->
+    <xacro:macro name="camera_xacro" params="xyz parent_link:=base_link rpy:='0 0 0' prefix:=camera">
         <!-- ============相机模块 - 缩小一半的小正方体================ -->
-        <link name="camera_link">
+        <link name="${prefix}_link">
             <visual>
                 <origin xyz="0 0 0.0" rpy="0 0 0" />
@@ -9,5 +10,5 @@
                     <box size="0.0125 0.0125 0.0125" />
                 </geometry>
-                <material name="red">
+                <material name="${prefix}_red">
                     <color rgba="1.0 0.0 0.0 1.0"/>
                 </material>
@@ -18,5 +19,5 @@
                     <box size="0.0125 0.0125 0.0125" />
                 </geometry>
-                <material name="red">
+                <material name="${prefix}_red">
                     <color rgba="1.0 0.0 0.0 1.0"/>
                 </material>
@@ -24,13 +25,13 @@
             <xacro:box_inertia m="0.0025" w="0.0125" h="0.0125" d="0.0125" />
         </link>
-        <link name="camera_optical_link"></link>
-        <joint name="camera_optical_joint" type="fixed">
-            <parent link="camera_link" />
-            <child link="camera_optical_link" />
+        <link name="${prefix}_optical_link"></link>
+        <joint name="${prefix}_optical_joint" type="fixed">
+            <parent link="${prefix}_link" />
+            <child link="${prefix}_optical_link" />
             <origin xyz="0 0 0" rpy="${-pi/2} 0 ${-pi/2}" />
         </joint>
-        <joint name="camera_joint" type="fixed">
+        <joint name="${prefix}_joint" type="fixed">
             <parent link="${parent_link}" />
-            <child link="camera_link" />
+            <child link="${prefix}_link" />
             <origin xyz="${xyz}" rpy="${rpy}" />
         </joint>
